Commit message: backkup

File: src/qcar_gazebo/urdf/camera.xacro (robot description, xacro)
@@ -6,9 +6,9 @@
             <update_rate>10</update_rate>
             <camera name="front">
-                <horizontal_fov>1.089</horizontal_fov>
+                <horizontal_fov>1.2043</horizontal_fov>
                 <image>
                 	<format>R8G8B8</format>
-                    <width>640</width>
-                    <height>480</height>
+                    <width>1280</width>
+                    <height>720</height>
                 </image>
             </camera>
@@ -26,6 +26,6 @@
                 <image>
                     <format>R8G8B8</format>
-                    <width>640</width>
-                    <height>480</height>
+                    <width>1280</width>
+                    <height>720</height>
                 </image>
             </camera>
@@ -43,6 +43,6 @@
                 <image>
                     <format>R8G8B8</format>
-                    <width>640</width>
-                    <height>480</height>
+                    <width>1280</width>
+                    <height>720</height>
                 </image>
             </camera>
@@ -60,6 +60,6 @@
                 <image>
                     <format>R8G8B8</format>
-                    <width>640</width>
-                    <height>480</height>
+                    <width>1280</width>
+                    <height>720</height>
                 </image>
             </camera>
@@ -79,6 +79,6 @@
         <image>
           <format>R8G8B8</format>
-          <width>640</width>
-          <height>480</height>
+          <width>1280</width>
+          <height>720</height>
         </image>
       </camera>

File: src/qcar_gazebo/urdf/depth_camera.xacro (robot description, xacro)
@@ -10,13 +10,13 @@
       <camera name="rgbd_front_depth_intrinsics">
         <!-- Match the color camera exactly for 1:1 pixel alignment -->
-        <horizontal_fov>1.089</horizontal_fov>
+        <horizontal_fov>1.5184</horizontal_fov>
         <image>
           <format>R8G8B8</format>
-          <width>640</width>
+          <width>848</width>
           <height>480</height>
         </image>
         <depth>
           <image>
-            <width>640</width>
+            <width>848</width>
             <height>480</height>
             <!-- IMPORTANT: publish float depth so ROS gets 32FC1 (meters) -->

File: src/qcar_gazebo/urdf/qcar_model.xacro (robot description, xacro)
@@ -247,4 +247,14 @@
   	</joint>
     <link name="camera_rgb"/>
+    <!-- ROS optical frame for the front RGBD camera
+         REP 105: Z forward, X right, Y down -->
+    <link name="rgbd_front_optical"/>
+    <joint name="rgbd_front_optical_joint" type="fixed">
+      <parent link="camera_rgb"/>
+      <child link="rgbd_front_optical"/>
+      <!-- Rotate camera_rgb into optical convention:
+           R = RotX(-90deg) * RotZ(-90deg) -->
+      <origin xyz="0 0 0" rpy="-1.57079632679 0 -1.57079632679"/>
+    </joint>
     <joint name="camera_csi_front_joint" type="fixed">
         <!-- <axis xyz="0 1 0" /> -->

Commit message: working but needs tuning with CSI

File: src/qcar_gazebo/urdf/camera.xacro (robot description, xacro)
@@ -1,18 +1,21 @@
 <?xml version='1.0'?>
 <robot xmlns:xacro="http://www.ros.org/wiki/xacro">
-	 <gazebo reference="camera_csi_front">
+   <gazebo reference="camera_csi_front">
         <sensor type="camera" name="front_camera">
-        	<visualize>true</visualize>
+            <visualize>true</visualize>
             <update_rate>10</update_rate>
             <camera name="front">
                 <horizontal_fov>1.2043</horizontal_fov>
                 <image>
-                	<format>R8G8B8</format>
+                    <format>R8G8B8</format>
                     <width>1280</width>
                     <height>720</height>
                 </image>
             </camera>
-            <plugin name="camera_controller" filename="libgazebo_ros_camera.so">
-                <cameraName>front_camera</cameraName>
+            <plugin name="camera_controller_front" filename="libgazebo_ros_camera.so">
+                <cameraName>csi_front</cameraName>
+                <frameName>csi_front_optical</frameName>
+                <imageTopicName>image_raw</imageTopicName>
+                <cameraInfoTopicName>camera_info</cameraInfoTopicName>
             </plugin>
         </sensor>
@@ -30,6 +33,9 @@
                 </image>
             </camera>
-            <plugin name="camera_controller" filename="libgazebo_ros_camera.so">
-                <cameraName>right_camera</cameraName>
+            <plugin name="camera_controller_right" filename="libgazebo_ros_camera.so">
+                <cameraName>csi_right</cameraName>
+                <frameName>csi_right_optical</frameName>
+                <imageTopicName>image_raw</imageTopicName>
+                <cameraInfoTopicName>camera_info</cameraInfoTopicName>
             </plugin>
         </sensor>
@@ -47,6 +53,9 @@
                 </image>
             </camera>
-            <plugin name="camera_controller" filename="libgazebo_ros_camera.so">
-                <cameraName>left_camera</cameraName>
+            <plugin name="camera_controller_left" filename="libgazebo_ros_camera.so">
+                <cameraName>csi_left</cameraName>
+                <frameName>csi_left_optical</frameName>
+                <imageTopicName>image_raw</imageTopicName>
+                <cameraInfoTopicName>camera_info</cameraInfoTopicName>
             </plugin>
         </sensor>
@@ -64,10 +73,10 @@
                 </image>
             </camera>
-            <plugin name="camera_controller" filename="libgazebo_ros_camera.so">
+            <plugin name="camera_controller_back" filename="libgazebo_ros_camera.so">
                 <cameraName>back_camera</cameraName>
             </plugin>
         </sensor>
     </gazebo>
-    <!-- NEW: RGB stream for the RGB-D head on the same link as the depth sensor -->
+    <!-- RGB stream for the RGB-D head (unchanged) -->
   <gazebo reference="camera_rgb">
     <sensor type="camera" name="rgbd_front_color">
@@ -75,5 +84,4 @@
       <update_rate>15</update_rate>
       <camera name="rgbd_front_color_intrinsics">
-        <!-- Match depth sensor settings 1:1 -->
         <horizontal_fov>1.211</horizontal_fov>
         <image>
@@ -84,9 +92,6 @@
       </camera>
       <plugin name="rgbd_color_controller" filename="libgazebo_ros_camera.so">
-        <!-- Same head name as depth -->
         <cameraName>rgbd_front</cameraName>
-        <!-- Share the exact same optical frame -->
         <frameName>rgbd_front_optical</frameName>
-        <!-- Own the main color topics -->
         <imageTopicName>image_raw</imageTopicName>
         <cameraInfoTopicName>camera_info</cameraInfoTopicName>

File: src/qcar_gazebo/urdf/qcar_model.xacro (robot description, xacro)
@@ -247,32 +247,37 @@
   	</joint>
     <link name="camera_rgb"/>
-    <!-- ROS optical frame for the front RGBD camera
-         REP 105: Z forward, X right, Y down -->
     <link name="rgbd_front_optical"/>
     <joint name="rgbd_front_optical_joint" type="fixed">
-      <parent link="camera_rgb"/>
-      <child link="rgbd_front_optical"/>
-      <!-- Rotate camera_rgb into optical convention:
-           R = RotX(-90deg) * RotZ(-90deg) -->
-      <origin xyz="0 0 0" rpy="-1.57079632679 0 -1.57079632679"/>
-    </joint>
+        <parent link="camera_rgb"/>
+        <child link="rgbd_front_optical"/>
+        <origin xyz="0 0 0" rpy="-1.57079632679 0 -1.57079632679"/>
+    </joint>
+    <!-- CSI FRONT -->
     <joint name="camera_csi_front_joint" type="fixed">
-        <!-- <axis xyz="0 1 0" /> -->
-        <!-- <origin xyz=".2 0 0" rpy="0 0 0"/> -->
         <origin rpy="0 0 0" xyz="0.19236 -0.000475 0.093029"/>
-        <!-- <origin rpy="0 0 0" xyz="0 0 0"/> -->
         <parent link="base"/>
         <child link="camera_csi_front"/>
     </joint>
     <link name="camera_csi_front"/>
+    <!-- Optical frame: REP 105 (Z forward, X right, Y down) -->
+    <link name="csi_front_optical"/>
+    <joint name="csi_front_optical_joint" type="fixed">
+        <parent link="camera_csi_front"/>
+        <child  link="csi_front_optical"/>
+        <origin xyz="0 0 0" rpy="-1.57079632679 0 -1.57079632679"/>
+    </joint>
+    <!-- CSI RIGHT -->
     <joint name="camera_csi_right_joint" type="fixed">
-        <!-- <axis xyz="0 1 0" /> -->
-        <!-- <origin xyz=".2 0 0" rpy="0 0 0"/> -->
-        <origin rpy="0 0 -1.5708" xyz="0.12887 -0.06755 0.093029"/>
-        <!-- <origin rpy="0 0 0" xyz="0 0 0"/> -->
-        <parent link="base"/>
-        <child link="camera_csi_right"/>
-    </joint>
-    <link name="camera_csi_right"/>
+      <origin rpy="0 0 -1.5708" xyz="0.12887 -0.06755 0.093029"/>
+      <parent link="base"/>
+      <child link="camera_csi_right"/>
+     </joint>
+     <link name="camera_csi_right"/>
+     <link name="csi_right_optical"/>
+     <joint name="csi_right_optical_joint" type="fixed">
+       <parent link="camera_csi_right"/>
+       <child  link="csi_right_optical"/>
+       <origin xyz="0 0 0" rpy="-1.57079632679 0 -1.57079632679"/>
+     </joint>
     <joint name="camera_csi_back_joint" type="fixed">
         <!-- <axis xyz="0 1 0" /> -->
@@ -284,13 +289,17 @@
     </joint>
     <link name="camera_csi_back"/>
+    <!-- CSI LEFT -->
     <joint name="camera_csi_left_joint" type="fixed">
-        <!-- <axis xyz="0 1 0" /> -->
-        <!-- <origin xyz=".2 0 0" rpy="0 0 0"/> -->
-        <origin rpy="0 0 1.5708" xyz="0.12784 0.052497 0.093029"/>
-        <!-- <origin rpy="0 0 0" xyz="0 0 0"/> -->
-        <parent link="base"/>
-        <child link="camera_csi_left"/>
+      <origin rpy="0 0 1.5708" xyz="0.12784 0.052497 0.093029"/>
+      <parent link="base"/>
+      <child link="camera_csi_left"/>
     </joint>
     <link name="camera_csi_left"/>
+    <link name="csi_left_optical"/>
+    <joint name="csi_left_optical_joint" type="fixed">
+        <parent link="camera_csi_left"/>
+        <child  link="csi_left_optical"/>
+        <origin xyz="0 0 0" rpy="-1.57079632679 0 -1.57079632679"/>
+    </joint>
     <transmission name="body_lidar_tran">
         <type>>transmission_interface/SimpleTransmission</type>
